File: bomu/bomu.sch (KiCad schematic (older format))
At the start: 35 parts, among them U1 NRF52840-CKAA-R7

Commit message: Adding gerbers, and current work
Parts:
- removed C_RF2: DNP, Capacitor_SMD:C_0201_0603Metric, symbol Device:C_Small
- removed L3: DNP, Inductor_SMD:L_0201_0603Metric, symbol Device:L
Connections:
- net at ANT1.FEED: now also C_RF1.1, L2.1
Changed lines of the file:
@@
 	900  4500 900  4700
-$Comp
-L Device:L L3
-U 1 1 5FEBFB1D
-P 9750 2800
-F 0 "L3" V 9940 2800 50  0000 C CNN
-F 1 "DNP" V 9849 2800 50  0000 C CNN
-F 2 "Inductor_SMD:L_0201_0603Metric" H 9750 2800 50  0001 C CNN
-F 3 "~" H 9750 2800 50  0001 C CNN
-	1    9750 2800
-	0    1    -1   0
-$EndComp
 $Comp
 L Device:C_Small C_RF1
@@
 	-1   0    0    -1
 $EndComp
-$Comp
-L Device:C_Small C_RF2
-U 1 1 5FEC1A7E
-P 9950 3000
-F 0 "C_RF2" H 10042 3046 50  0000 L CNN
-F 1 "DNP" H 10042 2955 50  0000 L CNN
-F 2 "Capacitor_SMD:C_0201_0603Metric" H 9950 3000 50  0001 C CNN
-F 3 "~" H 9950 3000 50  0001 C CNN
-	1    9950 3000
-	-1   0    0    -1
-$EndComp
 Wire Wire Line
 	9350 2800 9550 2800
 Wire Wire Line
-	9900 2800 9950 2800
-Wire Wire Line
 	9550 2900 9550 2800
 Connection ~ 9550 2800
-Wire Wire Line
-	9550 2800 9600 2800
-Wire Wire Line
-	9950 2900 9950 2800
-Connection ~ 9950 2800
-Wire Wire Line
-	9950 2800 10450 2800
 $Comp
 L power:GND #PWR0128
@@
 	-1   0    0    -1
 $EndComp
-$Comp
-L power:GND #PWR0129
-U 1 1 5FECDCAD
-P 9950 3200
-F 0 "#PWR0129" H 9950 2950 50  0001 C CNN
-F 1 "GND" H 9955 3027 50  0000 C CNN
-F 2 "" H 9950 3200 50  0001 C CNN
-F 3 "" H 9950 3200 50  0001 C CNN
-	1    9950 3200
-	-1   0    0    -1
-$EndComp
 Wire Wire Line
 	9550 3100 9550 3200
-Wire Wire Line
-	9950 3100 9950 3200
 $Comp
 L Connector:TestPoint TP9
@@
 Text Label 4650 3300 0    50   ~ 0
 P0.05
+Wire Wire Line
+	9550 2800 10450 2800
 $EndSCHEMATC

Commit message: Latest changes to the schematic and pcb
Parts:
- added C_RF2, C_RF3: DNP, Capacitor_SMD:C_0201_0603Metric, symbol Device:C_Small
- added L3: DNP, Inductor_SMD:L_0201_0603Metric, symbol Device:L
- added TP11, TP12: DNP, TestPoint:TestPoint_Pad_D1.0mm, symbol Connector:TestPoint
- ANT1: MP (none) -> W3008
- C1: MP (none) -> GRM0335C1E1R0BA01D
- C10, C8, C9: footprint Capacitor_SMD:C_0201_0603Metric -> Capacitor_SMD:C_0402_1005Metric; MP (none) -> C1005X5R1A475K050BC
- C11, C15: footprint Capacitor_SMD:C_0201_0603Metric -> Capacitor_SMD:C_0402_1005Metric; MP (none) -> 04026C105KAT2A
- C12, C13, C14, C2: MP (none) -> CL21B104KBFNNNG
- C3: MP (none) -> GRM033R71E821KA01D
- C4, C5: value C_Small -> 12pF; MP (none) -> GRM0335C1E120FA01J
- C6, C7: value C_Small -> 6pF; MP (none) -> GRM0335C1E6R0DA01D
- L1: MP (none) -> 0201DS-3N9XJEW
- L2: MP (none) -> LQP03PN4N7J02D
- R1: MP (none) -> RC0201FR-074R7L
- TP1, TP10, TP3, TP4, TP5, TP6, TP7, TP8, TP9: value TestPoint -> DNP
- U1: MP (none) -> NRF52840-CKAA-R7
- USB1: value USB-A-INSERT -> DNP
- XTAL1: DESCRIPTION 26MHz ±20ppm Crystal 10pF 100 Ohms 4-SMD, No Lead -> 32MHz ±20ppm Crystal 10pF 100 Ohms 4-SMD, No Lead
- XTAL2: MP (none) -> ABS06-107-32.768KHZ-T
Connections:
- net GND: now also C_RF2.2, C_RF3.2
- net at C_RF1.1, L2.1: now also L3.2; no longer ANT1.FEED
- net NFC-: now reaches U1.E2 (P0.10/NFC2)
- net NFC-: now also TP12.1
- net NFC+: now reaches U1.F1 (P0.09/NFC1)
- net NFC+: now also TP11.1
- new net: ANT1.FEED, C_RF2.1, C_RF3.1, L3.1

Commit message: Tonight's work on bomu. Added LC filter to VDD3P3 pins
Parts:
- C12, C13, C14, C2: MP CL21B104KBFNNNG -> GRM033R61E104KE14D
Changed lines of the file:
@@
 F 2 "Capacitor_SMD:C_0201_0603Metric" H 4700 6950 50  0001 C CNN
 F 3 "~" H 4700 6950 50  0001 C CNN
-F 4 "CL21B104KBFNNNG" H 4700 6950 50  0001 C CNN "MP"
+F 4 "GRM033R61E104KE14D" H 4700 6950 50  0001 C CNN "MP"
 	1    4700 6950
 	-1   0    0    1
@@
 F 2 "Capacitor_SMD:C_0201_0603Metric" H 4850 6950 50  0001 C CNN
 F 3 "~" H 4850 6950 50  0001 C CNN
-F 4 "CL21B104KBFNNNG" H 4850 6950 50  0001 C CNN "MP"
+F 4 "GRM033R61E104KE14D" H 4850 6950 50  0001 C CNN "MP"
 	1    4850 6950
 	1    0    0    -1
@@
 F 2 "Capacitor_SMD:C_0201_0603Metric" H 5150 7200 50  0001 C CNN
 F 3 "~" H 5150 7200 50  0001 C CNN
-F 4 "CL21B104KBFNNNG" H 5150 7200 50  0001 C CNN "MP"
+F 4 "GRM033R61E104KE14D" H 5150 7200 50  0001 C CNN "MP"
 	1    5150 7200
 	1    0    0    -1
@@
 F 2 "Capacitor_SMD:C_0201_0603Metric" H 1100 6850 50  0001 C CNN
 F 3 "~" H 1100 6850 50  0001 C CNN
-F 4 "CL21B104KBFNNNG" H 1100 6850 50  0001 C CNN "MP"
+F 4 "GRM033R61E104KE14D" H 1100 6850 50  0001 C CNN "MP"
 	1    1100 6850
 	1    0    0    -1

Commit message: Latest work on BOMU design
Parts:
- U1: MP NRF52840-CKAA-R7 -> NRF52840-CKAA-R
Changed lines of the file:
@@
 F 6 "0.514mm" H 6200 4100 50  0001 L BNN "MAXIMUM_PACKAGE_HEIGHT"
 F 7 "IPC7351B" H 6200 4100 50  0001 L BNN "STANDARD"
-F 8 "NRF52840-CKAA-R7" H 6200 4100 50  0001 C CNN "MP"
+F 8 "NRF52840-CKAA-R" H 6200 4100 50  0001 C CNN "MP"
 	1    6200 4100
 	1    0    0    -1
@@
 F 6 "0.514mm" H 3200 6700 50  0001 L BNN "MAXIMUM_PACKAGE_HEIGHT"
 F 7 "IPC7351B" H 3200 6700 50  0001 L BNN "STANDARD"
-F 8 "NRF52840-CKAA-R7" H 3200 6700 50  0001 C CNN "MP"
+F 8 "NRF52840-CKAA-R" H 3200 6700 50  0001 C CNN "MP"
 	2    3200 6700
 	1    0    0    -1
