File: bomu-programmer/bomu-programmer/bomu-programmer.kicad_sch (KiCad schematic)
At the start: 2 parts, among them J1 Conn_ARM_JTAG_SWD_10, P1 1mm_pitch_2x4

Commit message: Updating for KiCAD 7. Updated bomu-programmer board. Gerbers for bomu-programmer generated.
Parts:
- added J2: Conn_01x02, Connector_PinHeader_2.54mm:PinHeader_1x02_P2.54mm_Vertical, symbol Connector_Generic:Conn_01x02
Connections:
- net +3V3: now also J2.2 (Pin_2)
- net GND: now also J2.1 (Pin_1)
Changed lines of the file:
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@@
 (kicad_sch (version 20230121) (generator eeschema)
   (paper "A4")
+  (junction (at 78.74 78.74) (diameter 0) (color 0 0 0 0)
+  )
+  (junction (at 86.36 81.28) (diameter 0) (color 0 0 0 0)
+  )
   (junction (at 86.36 55.88) (diameter 0.9144) (color 0 0 0 0)
   )
@@
     (stroke (width 0) (type solid))
   )
+  (wire (pts (xy 86.36 81.28) (xy 147.32 81.28))
+    (stroke (width 0) (type default))
+  )
   (wire (pts (xy 87.63 39.37) (xy 87.63 22.86))
+    (stroke (width 0) (type solid))
+  )
+  (wire (pts (xy 78.74 78.74) (xy 78.74 99.06))
     (stroke (width 0) (type solid))
   )
@@
     (stroke (width 0) (type solid))
   )
+  (wire (pts (xy 78.74 78.74) (xy 147.32 78.74))
+    (stroke (width 0) (type default))
+  )
   (wire (pts (xy 49.53 163.83) (xy 59.69 163.83))
     (stroke (width 0) (type solid))
   )
-  (wire (pts (xy 86.36 55.88) (xy 86.36 87.63))
+  (wire (pts (xy 86.36 55.88) (xy 86.36 81.28))
     (stroke (width 0) (type solid))
   )
-  (wire (pts (xy 78.74 39.37) (xy 78.74 99.06))
+  (wire (pts (xy 78.74 39.37) (xy 78.74 78.74))
     (stroke (width 0) (type solid))
   )
@@
   )
   (wire (pts (xy 78.74 99.06) (xy 74.93 99.06))
+    (stroke (width 0) (type solid))
+  )
+  (wire (pts (xy 86.36 81.28) (xy 86.36 87.63))
     (stroke (width 0) (type solid))
   )
@@
         )
       )
+    )
+  )
+  (symbol (lib_id "Connector_Generic:Conn_01x02") (at 152.4 78.74 0) (unit 1)
+    (in_bom yes) (on_board yes) (dnp no) (fields_autoplaced)
+    (property "Reference" "J2" (at 154.94 79.375 0)
+      (effects (font (size 1.27 1.27)) (justify left))
+    )
+    (property "Value" "Conn_01x02" (at 154.94 81.915 0)
+      (effects (font (size 1.27 1.27)) (justify left))
+    )
+    (property "Footprint" "Connector_PinHeader_2.54mm:PinHeader_1x02_P2.54mm_Vertical" (at 152.4 78.74 0)
+      (effects (font (size 1.27 1.27)) hide)
+    )
+    (property "Datasheet" "~" (at 152.4 78.74 0)
+      (effects (font (size 1.27 1.27)) hide)
+    )
+    (pin "1")
+    (pin "2")
+    (instances
+      (project "bomu-programmer"
+        (path "/316cd380-1ab5-4859-81eb-60816364d980"
+          (reference "J2") (unit 1)
+        )
+      )
